File: Prova.brd (EAGLE design)
At the start: 41.9 x 48.6 mm, 32 parts, among them IC1 MAX31855, Q1 3904smd, Q2 3904smd

Commit message: minor bug fixes
Parts:
- removed LED: (no value), con-amp-quick:02P
- added R6: 10k, rcl:M0805
- moved U$2 20.3 mm to (6.99, 5.71), turned to 90 degrees
- moved R3 7.31 mm to (7.94, 15.9), turned to 0 degrees
- moved D1 4.14 mm to (11.7, 12.1)
- moved THERMOCOUPLE 0.64 mm to (9.84, 24.3)
Connections:
- net N$7 renamed VIN
- net +5V: now also R6.2; no longer R3.2
- net A0: now also R6.1
- net GND: now also R3.1
- net LED: now also D1.A; no longer D1.K, LED.2
- net N$6: now also D1.K, R3.2; no longer D1.A, LED.1, R3.1
Routing:
- net +5V: track 145.4 -> 112.6 mm
- net N$6: track 6.99 -> 2.54 mm
- net A0: track 15.2 -> 17.7 mm
- net LED: track 11.8 -> 10.4 mm
- net VIN: track 74.4 -> 73.5 mm
- net N$9: track 30.1 -> 30.7 mm
Other:
- board text removed: "C3"
- board text removed: "C4"
- board text removed: "FB1"
- board text removed: "FB2"
- board text removed: "R4"
- board text removed: "R5"
