File: Prova.sch (EAGLE design)
At the start: 29 parts, among them IC1 MAX31855, Q1 3904smd, Q2 3904smd

Commit message: minor bug fixes
Parts:
- removed LED: (no value), con-amp-quick:M02
- added R6: 10k, rcl:R-EU_M0805
Connections:
- net N$7 renamed VIN
- net +5V: now also R6.2; no longer R3.2
- net A0: now also R6.1
- net GND: now also R3.1
- net LED: now also D1.A; no longer D1.C, LED.2
- net N$6: now also D1.C, R3.2; no longer D1.A, LED.1, R3.1
Other:
- moved on the sheet: D1, R3
