File: Eagle/v2_zero/Arduino_Zero.sch (EAGLE design)
At the start: 71 parts, among them IC1 74HC125D, IC2 MAX31855, IC3 MAX31855, IC4 REG1117, IC5 ATSAMD21G-A, IC6 SPX3819-3.3, IC7 TXS0108E, IC8 TLP283, J3 USB-MICROB, J4 NM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

Commit message: update 3d packages
small updates
Parts:
- removed C18: 1uF, rcl:C-EUC0603K
- removed C20: 4.7uF, rcl:C-EUC0603K
- added C3, C9: TAJB106K020RNJ, microbuilder:CAP_TANTALUM
- IC8: device optocoupler:TLP283 -> gfe-hand-made:TLP292
Connections:
- net +5V: now also C9.+; no longer C20.1
- net 12V: now also C3.+; no longer C18.1
- net GND: now also C3.-, C9.-, IC8.3; no longer C18.2, C20.2, IC8.C, IC8.EMIT
- net N$12: no longer IC8.A
- net N$14: now also IC8.4; no longer IC8.COL
Other:
- moved on the sheet: J5-1, J5-2, Q3, R10

Commit message: schematic update
Parts:
- removed C6, C7: 10uF, rcl:C-EUC0603K
- removed D2, D4, D5, D6: 1N4148, adafruit:DIODESOD-323-3D
- removed R14, R15, R8, R9: 10K, rcl:R-EU_R0603
- removed SV1: (no value), con-lstb:MA03-1
- added J9: (no value), adafruit:PINHD-1X3
Connections:
- removed net CS1: D4.A, IC3./CS, R15.2
- removed net CS2: D6.A, IC2./CS, R9.2
- removed net SCK1: D5.A, IC2.SCK, R8.2
- removed net SCK2: D2.A, IC3.SCK, R14.2
- net +3V3: no longer C6.1, C7.1, R14.1, R15.1, R8.1, R9.1
- net +5V: now also J9.3; no longer SV1.3
- net A1_BTN: now also J9.2; no longer SV1.2
- net A2_TC1_CS: now also IC2./CS; no longer D6.C
- net A3_TC2_CS: now also IC3./CS; no longer D4.C
- net GND: now also IC8.2, J9.1; no longer C6.2, C7.2, SV1.1
- net N$12: now also IC8.1
- net SCK: now also IC2.SCK, IC3.SCK; no longer D2.C, D5.C
Other:
- moved on the sheet: C2

Commit message: schematic optimization
Parts:
- C1, C2: value 10uF -> 100n
Connections:
- net N$29 renamed XIN32
- net N$31 renamed XOUT32
Changed lines of the file:
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@@
 <part name="U$18" library="microbuilder" deviceset="12V" device=""/>
 <part name="GND10" library="supply1" library_urn="urn:adsk.eagle:library:371" deviceset="GND" device=""/>
-<part name="C1" library="rcl" library_urn="urn:adsk.eagle:library:334" deviceset="C-EU" device="C0603K" package3d_urn="urn:adsk.eagle:package:23680/2" value="10uF"/>
+<part name="C1" library="rcl" library_urn="urn:adsk.eagle:library:334" deviceset="C-EU" device="C0603K" package3d_urn="urn:adsk.eagle:package:23680/2" value="100n"/>
 <part name="IC3" library="adafruit" deviceset="MAX6675" device="" override_package3d_urn="urn:adsk.eagle:package:35728084/2" override_package_urn="urn:adsk.eagle:footprint:35728085/1" value="MAX31855"/>
 <part name="GND11" library="supply1" library_urn="urn:adsk.eagle:library:371" deviceset="GND" device=""/>
 <part name="+3V17" library="supply1" library_urn="urn:adsk.eagle:library:371" deviceset="+3V3" device=""/>
 <part name="+3V18" library="supply1" library_urn="urn:adsk.eagle:library:371" deviceset="+3V3" device=""/>
-<part name="C2" library="rcl" library_urn="urn:adsk.eagle:library:334" deviceset="C-EU" device="C0603K" package3d_urn="urn:adsk.eagle:package:23680/2" value="10uF"/>
+<part name="C2" library="rcl" library_urn="urn:adsk.eagle:library:334" deviceset="C-EU" device="C0603K" package3d_urn="urn:adsk.eagle:package:23680/2" value="100n"/>
 <part name="+3V19" library="supply1" library_urn="urn:adsk.eagle:library:371" deviceset="+3V3" device=""/>
 <part name="GND19" library="supply1" library_urn="urn:adsk.eagle:library:371" deviceset="GND" device=""/>
@@
 </segment>
 </net>
-<net name="N$29" class="0">
+<net name="XIN32" class="0">
 <segment>
 <pinref part="C12" gate="G$1" pin="1"/>
@@
 <wire x1="332.74" y1="76.2" x2="350.52" y2="76.2" width="0.1524" layer="91"/>
 <wire x1="332.74" y1="81.28" x2="332.74" y2="76.2" width="0.1524" layer="91"/>
-</segment>
-</net>
-<net name="N$31" class="0">
+<label x="337.82" y="76.2" size="1.778" layer="95"/>
+</segment>
+</net>
+<net name="XOUT32" class="0">
 <segment>
 <pinref part="C11" gate="G$1" pin="1"/>
@@
 <pinref part="IC5" gate="G$1" pin="PA01(XOUT32/SER1:1/TC2:1)"/>
 <wire x1="332.74" y1="71.12" x2="350.52" y2="71.12" width="0.1524" layer="91"/>
-</segment>
-</net>
+<label x="337.82" y="71.12" size="1.778" layer="95"/>
+</segment>
+</net>

Commit message: update
Parts:
- removed IC6: SPX3819-3.3, microbuilder:VREG_SOT23-5
- removed R6: 100k, rcl:R-EU_R0603
- added IC9: REG1117-5, gfe-hand-made:REG1117-5
- C5: value 2.2 µF -> TAJB106K020RNJ; device Wurth_Capacitors_WCAP-ASLI:WCAP-ASLI_4X5.5_865080640002 -> microbuilder:CAP_TANTALUM
- IC4: value REG1117 -> REG1117-3.3; device burr-brown:REG1117 -> gfe-hand-made:REG1117-5
- R3: value (none) -> 470R
- R7: value (none) -> 10k
Connections:
- net D0_RX renamed !ETH_RST
- net D12 renamed ETH_CS
- net D1_TX renamed ETH_IRQ
- removed net EN: IC6.EN, R6.2
- net +3V3: now also IC4.VOUT2, IC4.VOUT4; no longer IC6.OUT
- net +5V: now also IC4.IN, IC9.VOUT2, IC9.VOUT4; no longer IC4.VOUT, IC6.IN, R6.1
- net 12V: now also IC9.IN; no longer IC4.VIN
- net GND: now also IC9.GND; no longer IC6.GND
Other:
- moved on the sheet: C21, R11, R12, SJ1
